File: panel.sch (KiCad schematic (older format))
At the start: 1 part, among them U1 led-panel-16x16

Commit message: Finish STM32 digital interface assignment
Connections:
- wire segments 197 -> 176
Changed lines of the file:
@@
 $Descr A4 11693 8268
 encoding utf-8
-Sheet 10 24
+Sheet 2 25
 Title ""
 Date ""
@@
 AR Path="/61C4C20D/61A429F9" Ref="U9"  Part="1"
 AR Path="/61C4C905/61A429F9" Ref="U16"  Part="1"
-F 0 "U16" H 3625 6915 50  0000 C CNN
+F 0 "U1" H 3625 6915 50  0000 C CNN
 F 1 "led-panel-16x16" H 3625 6824 50  0000 C CNN
 F 2 "led-panel:bga-led-panel-16x16" H 3400 6800 50  0001 C CNN
@@
 R9
 Wire Wire Line
-	1600 1600 1450 1600
-Text Label 1450 1600 0    50   ~ 0
-R2
-Wire Wire Line
-	1600 1500 1450 1500
-Text Label 1450 1500 0    50   ~ 0
-G2
-Wire Wire Line
-	1600 1400 1450 1400
-Text Label 1450 1400 0    50   ~ 0
-B2
-Wire Wire Line
 	4900 1450 4750 1450
 Text Label 4750 1450 0    50   ~ 0
@@
 B4
 Wire Wire Line
-	1600 1700 1450 1700
-Text Label 1450 1700 0    50   ~ 0
-G6
-Wire Wire Line
-	1600 1800 1450 1800
-Text Label 1450 1800 0    50   ~ 0
-R6
-Wire Wire Line
-	1600 2900 1450 2900
-Text Label 1450 2900 0    50   ~ 0
-B6
-Wire Wire Line
-	1600 2800 1450 2800
-Text Label 1450 2800 0    50   ~ 0
-R8
-Wire Wire Line
-	1600 2700 1450 2700
-Text Label 1450 2700 0    50   ~ 0
-G8
-Wire Wire Line
-	1600 2600 1450 2600
-Text Label 1450 2600 0    50   ~ 0
-B8
-Wire Wire Line
-	1600 2200 1450 2200
-Text Label 1450 2200 0    50   ~ 0
-R12
-Wire Wire Line
-	1600 2300 1450 2300
-Text Label 1450 2300 0    50   ~ 0
-B10
-Wire Wire Line
-	1600 2400 1450 2400
-Text Label 1450 2400 0    50   ~ 0
-G10
-Wire Wire Line
-	1600 2500 1450 2500
-Text Label 1450 2500 0    50   ~ 0
-R10
-Wire Wire Line
-	1600 3550 1450 3550
-Text Label 1450 3550 0    50   ~ 0
-B16
-Wire Wire Line
-	1600 3650 1450 3650
-Text Label 1450 3650 0    50   ~ 0
-G16
-Wire Wire Line
-	1600 3750 1450 3750
-Text Label 1450 3750 0    50   ~ 0
-R16
-Wire Wire Line
-	1600 3250 1450 3250
-Text Label 1450 3250 0    50   ~ 0
-R14
-Wire Wire Line
-	1600 3150 1450 3150
-Text Label 1450 3150 0    50   ~ 0
-G14
-Wire Wire Line
-	1600 3850 1450 3850
-Text Label 1450 3850 0    50   ~ 0
-B14
-Wire Wire Line
-	1600 3450 1450 3450
-Text Label 1450 3450 0    50   ~ 0
-G12
-Wire Wire Line
-	1600 3350 1450 3350
-Text Label 1450 3350 0    50   ~ 0
-B12
-Wire Wire Line
 	4900 1750 4750 1750

Commit message: Route ESP32 SPI bus
Changed lines of the file:
@@
 AR Path="/61C4C20D/61A429F9" Ref="U9"  Part="1"
 AR Path="/61C4C905/61A429F9" Ref="U16"  Part="1"
-F 0 "U1" H 3625 6915 50  0000 C CNN
+F 0 "U16" H 3625 6915 50  0000 C CNN
 F 1 "led-panel-16x16" H 3625 6824 50  0000 C CNN
 F 2 "led-panel:bga-led-panel-16x16" H 3400 6800 50  0001 C CNN

Commit message: Add 16MHz crystal
Turns out the STM32F7 DFU bootloader uses the HSE for USB clocking and
thus requires a crystal. No fallback to HSI is implemented. *sigh*
Changed lines of the file:
@@
 $Descr A4 11693 8268
 encoding utf-8
-Sheet 2 25
+Sheet 10 25
 Title ""
 Date ""
@@
 AR Path="/61C4C20D/61A429F9" Ref="U9"  Part="1"
 AR Path="/61C4C905/61A429F9" Ref="U16"  Part="1"
-F 0 "U16" H 3625 6915 50  0000 C CNN
+F 0 "U9" H 3625 6915 50  0000 C CNN
 F 1 "led-panel-16x16" H 3625 6824 50  0000 C CNN
 F 2 "led-panel:bga-led-panel-16x16" H 3400 6800 50  0001 C CNN

Commit message: Make space for STM32
Changed lines of the file:
@@
 $Descr A4 11693 8268
 encoding utf-8
-Sheet 10 25
+Sheet 2 25
 Title ""
 Date ""
@@
 AR Path="/61C4C20D/61A429F9" Ref="U9"  Part="1"
 AR Path="/61C4C905/61A429F9" Ref="U16"  Part="1"
-F 0 "U9" H 3625 6915 50  0000 C CNN
+F 0 "U1" H 3625 6915 50  0000 C CNN
 F 1 "led-panel-16x16" H 3625 6824 50  0000 C CNN
 F 2 "led-panel:bga-led-panel-16x16" H 3400 6800 50  0001 C CNN

Commit message: Add tag connect programming/debug interface
Changed lines of the file:
@@
 $Descr A4 11693 8268
 encoding utf-8
-Sheet 2 25
+Sheet 17 25
 Title ""
 Date ""
@@
 AR Path="/61C4C20D/61A429F9" Ref="U9"  Part="1"
 AR Path="/61C4C905/61A429F9" Ref="U16"  Part="1"
-F 0 "U1" H 3625 6915 50  0000 C CNN
+F 0 "U16" H 3625 6915 50  0000 C CNN
 F 1 "led-panel-16x16" H 3625 6824 50  0000 C CNN
 F 2 "led-panel:bga-led-panel-16x16" H 3400 6800 50  0001 C CNN
